File: ESP32-SPI.kicad_pcb (KiCad board)
At the start: 2 copper layers, 35 x 50 mm, 3 parts, among them J1 SPI-Connector

Commit message: Add files via upload
Parts:
- J1: footprint Connector_Samtec_HLE_THT:Samtec_HLE-105-02-xx-DV-TE_2x05_P2.54mm_Horizontal -> Connector_PinSocket_2.54mm:PinSocket_2x05_P2.54mm_Vertical
- turned J1 to 90 degrees
Connections:
- net /11-INT renamed /6-INT
- net /12-MOSI renamed /7-MOSI
- net /13-RST renamed /8-RST
- net /16-MISO renamed /17-MISO
- net /21-SCS renamed /18-SCS
- H1 pad 2: /2-SCLK -> /2
- H1 pad 3: /3 -> /3-SCLK
- J1 pad 1: /2-SCLK -> /3-SCLK
- S1 pad 2: /2-SCLK -> /2
- S1 pad 3: /3 -> /3-SCLK
Routing:
- net /2-SCLK: track 20.6 -> 0.00 mm
- net /3-SCLK: track 0.00 -> 19.5 mm
- net /7-MOSI: track 35.3 -> 18.3 mm
- net /2: track 0.00 -> 6.09 mm
- net /3: track 6.05 -> 0.00 mm

Commit message: Add files via upload
Connections:
- H1 pad 4: /4 -> /4-RST
- H1 pad 6: /6-INT -> /6
- H1 pad 8: /8-RST -> /8
- J1 pad 4: /6-INT -> /4
- J1 pad 6: /8-RST -> /4-RST
- S1 pad 4: /4 -> /4-RST
- S1 pad 6: /6-INT -> /6
- S1 pad 8: /8-RST -> /8
Routing:
- net /4-RST: track 0.00 -> 19.5 mm
- net /8-RST: track 15.5 -> 0.00 mm
- net /6-INT: track 14.5 -> 0.00 mm
- net /6: track 0.00 -> 6.01 mm
- net /8: track 0.00 -> 6.00 mm
- net /4: track 6.00 -> 0.00 mm
