File: ESP32-SPI.kicad_sch (KiCad schematic)
At the start: 3 parts, among them J1 SPI-Connector

Commit message: Add files via upload
Parts:
- J1: footprint Connector_Samtec_HLE_THT:Samtec_HLE-105-02-xx-DV-TE_2x05_P2.54mm_Horizontal -> Connector_PinSocket_2.54mm:PinSocket_2x05_P2.54mm_Vertical
Connections:
- net 11-INT renamed 6-INT
- net 12-MOSI renamed 7-MOSI
- net 13-RST renamed 8-RST
- net 16-MISO renamed 17-MISO
- net 2-SCLK renamed 2
- net 2: no longer J1.1 (Pin_1)
- net 21-SCS renamed 18-SCS
- net 3 renamed 3-SCLK
- net 3-SCLK: now also J1.1 (Pin_1)
Changed lines of the file:
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@@
 		)
 	)
-	(label "13-RST"
+	(label "8-RST"
 		(at 115.57 34.29 270)
 		(effects
@@
 		)
 	)
-	(label "2-SCLK"
+	(label "2"
 		(at 83.82 34.29 270)
 		(effects
@@
 		)
 	)
-	(label "11-INT"
+	(label "6-INT"
 		(at 63.5 31.75 90)
 		(effects
@@
 		)
 	)
-	(label "2-SCLK"
+	(label "3-SCLK"
 		(at 71.12 31.75 90)
 		(effects
@@
 		)
 	)
-	(label "12-MOSI"
+	(label "7-MOSI"
 		(at 60.96 31.75 90)
 		(effects
@@
 		)
 	)
-	(label "16-MISO"
+	(label "17-MISO"
 		(at 63.5 55.88 270)
 		(effects
@@
 		)
 	)
-	(label "13-RST"
+	(label "8-RST"
 		(at 91.44 34.29 270)
 		(effects
@@
 		)
 	)
-	(label "11-INT"
+	(label "6-INT"
 		(at 113.03 34.29 270)
 		(effects
@@
 		)
 	)
-	(label "16-MISO"
+	(label "17-MISO"
 		(at 91.44 55.88 90)
 		(effects
@@
 		)
 	)
-	(label "12-MOSI"
+	(label "7-MOSI"
 		(at 114.3 34.29 270)
 		(effects
@@
 		)
 	)
-	(label "13-RST"
+	(label "8-RST"
 		(at 60.96 55.88 270)
 		(effects
@@
 		)
 	)
-	(label "12-MOSI"
+	(label "7-MOSI"
 		(at 90.17 34.29 270)
 		(effects
@@
 		)
 	)
-	(label "21-SCS"
+	(label "18-SCS"
 		(at 114.3 55.88 90)
 		(effects
@@
 		)
 	)
-	(label "16-MISO"
+	(label "17-MISO"
 		(at 115.57 55.88 90)
 		(effects
@@
 		)
 	)
-	(label "3"
+	(label "3-SCLK"
 		(at 85.09 34.29 270)
 		(effects
@@
 		)
 	)
-	(label "21-SCS"
+	(label "18-SCS"
 		(at 90.17 55.88 90)
 		(effects
@@
 		)
 	)
-	(label "3"
+	(label "3-SCLK"
 		(at 109.22 34.29 270)
 		(effects
@@
 		)
 	)
-	(label "2-SCLK"
+	(label "2"
 		(at 107.95 34.29 270)
 		(effects
@@
 		)
 	)
-	(label "11-INT"
+	(label "6-INT"
 		(at 88.9 34.29 270)
 		(effects
@@
 		)
 	)
-	(label "21-SCS"
+	(label "18-SCS"
 		(at 66.04 31.75 90)
 		(effects
@@
 			)
 		)
-		(property "Footprint" "Connector_Samtec_HLE_THT:Samtec_HLE-105-02-xx-DV-TE_2x05_P2.54mm_Horizontal"
+		(property "Footprint" "Connector_PinSocket_2.54mm:PinSocket_2x05_P2.54mm_Vertical"
 			(at 66.04 44.45 0)
 			(hide yes)

Commit message: Add files via upload
Connections:
- net 4: now also J1.4 (Pin_4); no longer H1.4 (GPIO3), S1.4 (GPIO3)
- net 6-INT renamed 6
- net 6: no longer J1.4 (Pin_4)
- net 8-RST renamed 8
- net 8: no longer J1.6 (Pin_6)
- new net 4-RST: H1.4 (GPIO3), J1.6 (Pin_6), S1.4 (GPIO3)
Changed lines of the file:
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@@
 		)
 	)
-	(label "8-RST"
+	(label "8"
 		(at 115.57 34.29 270)
 		(effects
@@
 		)
 	)
-	(label "6-INT"
+	(label "4"
 		(at 63.5 31.75 90)
 		(effects
@@
 		)
 	)
-	(label "8-RST"
+	(label "8"
 		(at 91.44 34.29 270)
 		(effects
@@
 		)
 	)
-	(label "4"
+	(label "4-RST"
 		(at 110.49 34.29 270)
 		(effects
@@
 		)
 	)
-	(label "6-INT"
+	(label "6"
 		(at 113.03 34.29 270)
 		(effects
@@
 		)
 	)
-	(label "8-RST"
+	(label "4-RST"
 		(at 60.96 55.88 270)
 		(effects
@@
 		)
 	)
-	(label "4"
+	(label "4-RST"
 		(at 86.36 34.29 270)
 		(effects
@@
 		)
 	)
-	(label "6-INT"
+	(label "6"
 		(at 88.9 34.29 270)
 		(effects
